File: ArduinoNameCard.sch (KiCad schematic (older format))
At the start: 24 parts, among them J2 Conn_01x04, J3 Conn_01x06, J4 Conn_01x08, J5 Conn_01x06, SW1 SW_Push, U2 MCU-ATMEGA328P-AU(TQFP32)

Commit message: FT232RLをFT230XSに置き換えた。
Parts:
- J1: renamed from J?; footprint (none) -> ArduinoNameCard:namecard_microB
- R2: renamed from R?; footprint (none) -> Resistors_SMD:R_0805_HandSoldering
- U1: renamed from U?; footprint (none) -> Housings_SSOP:SSOP-16_3.9x4.9mm_Pitch0.635mm
- renumbered C3 to C1, C1 to C2, C5 to C3
Connections:
- wire segments 139 -> 138
Changed lines of the file:
@@
 $EndComp
 $Comp
-L ArduinoNameCard-rescue:C- C3
+L ArduinoNameCard-rescue:C- C1
 U 1 1 598D8407
 P 1950 5500
-F 0 "C3" H 1975 5600 50  0000 L CNN
+F 0 "C1" H 1975 5600 50  0000 L CNN
 F 1 "0.1u" H 1975 5400 50  0000 L CNN
 F 2 "Capacitors_SMD:C_0805_HandSoldering" H 1988 5350 50  0001 C CNN
@@
 $EndComp
 $Comp
-L Device:C C1
+L Device:C C2
 U 1 1 598D853B
 P 2650 5500
-F 0 "C1" H 2675 5600 50  0000 L CNN
+F 0 "C2" H 2675 5600 50  0000 L CNN
 F 1 "0.1u" H 2675 5400 50  0000 L CNN
 F 2 "Capacitors_SMD:C_0805_HandSoldering" H 2688 5350 50  0001 C CNN
@@
 $EndComp
 $Comp
-L Device:C C5
+L Device:C C3
 U 1 1 598DE610
 P 6900 3650
-F 0 "C5" H 6925 3750 50  0000 L CNN
+F 0 "C3" H 6925 3750 50  0000 L CNN
 F 1 "22p" H 6925 3550 50  0000 L CNN
 F 2 "Capacitors_SMD:C_0805_HandSoldering" H 6938 3500 50  0001 C CNN
@@
 	1    0    0    -1
 $EndComp
-Text GLabel 2150 2500 2    60   Output ~ 0
+Text GLabel 2050 2500 3    60   Output ~ 0
 5V
 Wire Wire Line
 	2050 1950 2050 2050
-Wire Wire Line
-	2150 2500 2050 2500
 Wire Wire Line
 	2050 2500 2050 2350
@@
 	6950 2650 7550 2650
 $Comp
-L Connector:USB_B_Micro J?
+L Connector:USB_B_Micro J1
 U 1 1 5C66CF79
 P 3050 2200
-F 0 "J?" H 3105 2667 50  0000 C CNN
+F 0 "J1" H 3105 2667 50  0000 C CNN
 F 1 "USB_B_Micro" H 3105 2576 50  0000 C CNN
-F 2 "" H 3200 2150 50  0001 C CNN
+F 2 "ArduinoNameCard:namecard_microB" H 3200 2150 50  0001 C CNN
 F 3 "~" H 3200 2150 50  0001 C CNN
 	1    3050 2200
@@
 	3050 2600 3050 2700
 $Comp
-L ArduinoNameCard:FT230XS U?
+L ArduinoNameCard:FT230XS U1
 U 1 1 5C6C3281
 P 3550 4850
-F 0 "U?" H 3550 4950 50  0000 C CNN
+F 0 "U1" H 3550 4950 50  0000 C CNN
 F 1 "FT230XS" H 3550 4850 50  0000 C CNN
-F 2 "" H 3550 4550 50  0001 C CNN
+F 2 "Housings_SSOP:SSOP-16_3.9x4.9mm_Pitch0.635mm" H 3550 4550 50  0001 C CNN
 F 3 "https://www.ftdichip.com/Support/Documents/DataSheets/ICs/DS_FT230X.pdf" H 3550 4550 50  0001 C CNN
 	1    3550 4850
@@
 	2550 4650 2450 4650
 $Comp
-L power:GND #PWR?
+L power:GND #PWR0101
 U 1 1 5C75530E
 P 3450 5800
-F 0 "#PWR?" H 3450 5550 50  0001 C CNN
+F 0 "#PWR0101" H 3450 5550 50  0001 C CNN
 F 1 "GND" H 3455 5627 50  0000 C CNN
 F 2 "" H 3450 5800 50  0001 C CNN
@@
 Connection ~ 2650 4450
 $Comp
-L power:GND #PWR?
+L power:GND #PWR0102
 U 1 1 5C83D5A5
 P 2650 5800
-F 0 "#PWR?" H 2650 5550 50  0001 C CNN
+F 0 "#PWR0102" H 2650 5550 50  0001 C CNN
 F 1 "GND" H 2655 5627 50  0000 C CNN
 F 2 "" H 2650 5800 50  0001 C CNN
@@
 	4500 4350 4700 4350
 $Comp
-L Device:R R?
+L Device:R R2
 U 1 1 5C9978E4
 P 3650 2400
-F 0 "R?" V 3750 2400 50  0000 C CNN
+F 0 "R2" V 3750 2400 50  0000 C CNN
 F 1 "27" V 3650 2400 50  0000 C CNN
-F 2 "" V 3580 2400 50  0001 C CNN
+F 2 "Resistors_SMD:R_0805_HandSoldering" V 3580 2400 50  0001 C CNN
 F 3 "~" H 3650 2400 50  0001 C CNN
 	1    3650 2400

Commit message: FT231Xに変更した。
Parts:
- removed CP1: 10u, Capacitors_SMD:C_0805_HandSoldering, symbol ArduinoNameCard-rescue:CP-
- removed U1: FT230XS, Housings_SSOP:SSOP-16_3.9x4.9mm_Pitch0.635mm, symbol ArduinoNameCard:FT230XS
- added C5: 0.1u, Capacitors_SMD:C_0805_HandSoldering, symbol Device:C
- added R7: 10k, Resistors_SMD:R_0805_HandSoldering, symbol Device:R
- added U1: FT231XS, SMD_Packages:SSOP-20, symbol ArduinoNameCard:FT231XS
- D1: value RED -> RED(TX)
- D2: value GREEN -> GREEN(RX)
Connections:
- net labels added: DTR
- wire segments 138 -> 129
- no-connect marks 7 -> 11
Other:
- moved on the sheet: C2

Commit message: 部品の並びなどを修正した。
Parts:
- renumbered C5 to C3, C3 to C5, R7 to R5, R5 to R6, R6 to R7
Connections:
- net labels removed: RTS
Changed lines of the file:
@@
 $EndComp
 $Comp
-L Device:R R5
+L Device:R R6
 U 1 1 598DD49C
 P 6700 2250
-F 0 "R5" V 6780 2250 50  0000 C CNN
+F 0 "R6" V 6780 2250 50  0000 C CNN
 F 1 "10k" V 6700 2250 50  0000 C CNN
 F 2 "Resistors_SMD:R_0805_HandSoldering" V 6630 2250 50  0001 C CNN
@@
 $EndComp
 $Comp
-L Device:C C3
+L Device:C C5
 U 1 1 598DE610
 P 6900 3650
-F 0 "C3" H 6925 3750 50  0000 L CNN
+F 0 "C5" H 6925 3750 50  0000 L CNN
 F 1 "22p" H 6925 3550 50  0000 L CNN
 F 2 "Capacitors_SMD:C_0805_HandSoldering" H 6938 3500 50  0001 C CNN
@@
 $EndComp
 $Comp
-L Device:R R6
+L Device:R R7
 U 1 1 598E3542
 P 9800 5200
-F 0 "R6" V 9880 5200 50  0000 C CNN
+F 0 "R7" V 9880 5200 50  0000 C CNN
 F 1 "330" V 9800 5200 50  0000 C CNN
 F 2 "Resistors_SMD:R_0805_HandSoldering" V 9730 5200 50  0001 C CNN
@@
 $EndComp
 Text GLabel 4750 2100 0    60   Input ~ 0
-RTS
+DTR
 Wire Wire Line
 	7550 3250 7550 3350
@@
 	2550 4450 2550 4350
 $Comp
-L Device:R R7
+L Device:R R5
 U 1 1 5CED0EBC
 P 2550 5250
-F 0 "R7" V 2630 5250 50  0000 C CNN
+F 0 "R5" V 2630 5250 50  0000 C CNN
 F 1 "10k" V 2550 5250 50  0000 C CNN
 F 2 "Resistors_SMD:R_0805_HandSoldering" V 2480 5250 50  0001 C CNN
@@
 	1300 5300 1300 5550
 $Comp
-L Device:C C5
+L Device:C C3
 U 1 1 5CF1D9AE
 P 4900 4950
-F 0 "C5" H 4925 5050 50  0000 L CNN
+F 0 "C3" H 4925 5050 50  0000 L CNN
 F 1 "0.1u" H 4925 4850 50  0000 L CNN
 F 2 "Capacitors_SMD:C_0805_HandSoldering" H 4938 4800 50  0001 C CNN
